Commit message: added nav2 yaml and launch files

File: src/robot_description/urdf/qcar_model.xacro (robot description, xacro)
@@ -33,4 +33,21 @@
     </inertial>
   </link>
+  <!-- ====================== BASE FOOTPRINT ====================== -->
+  <!-- 2D navigation frame (no roll/pitch). Kept coincident with base for Nav2/SLAM -->
+  <link name="base_footprint"/>
+  <joint name="base_to_base_footprint" type="fixed">
+    <parent link="base"/>
+    <child link="base_footprint"/>
+    <origin xyz="0 0 0" rpy="0 0 0"/>
+  </joint>
+  <!-- ====================== BASE_LINK (Nav2 compatibility) ====================== -->
+  <!-- Keep 'base' as the real robot base, but also provide 'base_link' as an alias
+       because many Nav2 components default to base_link. -->
+  <link name="base_link"/>
+  <joint name="base_to_base_link" type="fixed">
+    <parent link="base"/>
+    <child link="base_link"/>
+    <origin xyz="0 0 0" rpy="0 0 0"/>
+  </joint>
   <!-- ====================== LIDAR ====================== -->
   <link name="lidar">

Commit message: simple ekf added, lidar and ekf works

File: src/robot_description/urdf/qcar_model.xacro (robot description, xacro)
@@ -1,340 +1,378 @@
-<?xml version="1.0"?>
-<robot name="QCar" xmlns:xacro="http://www.ros.org/wiki/xacro">
-  <!-- ====================== MATERIALS ====================== -->
-  <material name="black"><color rgba="0 0 0 1"/></material>
-  <material name="blue"><color rgba="0 0 0.8 1"/></material>
-  <material name="green"><color rgba="0 0.8 0 1"/></material>
-  <material name="grey"><color rgba="0.2 0.2 0.2 1"/></material>
-  <material name="orange"><color rgba="1.0 0.4235 0.0392 1"/></material>
-  <material name="brown"><color rgba="0.8706 0.8118 0.7647 1"/></material>
-  <material name="red"><color rgba="0.8 0 0 1"/></material>
-  <material name="white"><color rgba="1 1 1 1"/></material>
-  <!-- ====================== INCLUDES ====================== -->
-  <xacro:include filename="$(find realsense2_description)/urdf/_d435.urdf.xacro" />
-  <!-- ====================== BASE LINK ====================== -->
-  <link name="base">
-    <visual>
-      <origin xyz="0 0 0" rpy="0 0 0"/>
-      <geometry>
-        <mesh filename="package://robot_description/models/qcar/QCarBody.stl" scale="0.001 0.001 0.001"/>
-      </geometry>
-      <material name="white"/>
-    </visual>
-    <collision>
-      <origin xyz="0 0 0" rpy="0 0 0"/>
-      <geometry>
-        <mesh filename="package://robot_description/models/qcar/QCarBody.stl" scale="0.001 0.001 0.001"/>
-      </geometry>
-    </collision>
-    <inertial>
-      <origin xyz="0 0 0" rpy="0 0 0"/>
-      <mass value="0.1"/>
-      <inertia ixx="0.001" ixy="0" ixz="0" iyy="0.001" iyz="0" izz="0.001"/>
-    </inertial>
-  </link>
-  <!-- ====================== BASE FOOTPRINT ====================== -->
-  <!-- 2D navigation frame (no roll/pitch). Kept coincident with base for Nav2/SLAM -->
-  <link name="base_footprint"/>
-  <joint name="base_to_base_footprint" type="fixed">
-    <parent link="base"/>
-    <child link="base_footprint"/>
-    <origin xyz="0 0 0" rpy="0 0 0"/>
-  </joint>
-  <!-- ====================== BASE_LINK (Nav2 compatibility) ====================== -->
-  <!-- Keep 'base' as the real robot base, but also provide 'base_link' as an alias
-       because many Nav2 components default to base_link. -->
-  <link name="base_link"/>
-  <joint name="base_to_base_link" type="fixed">
-    <parent link="base"/>
-    <child link="base_link"/>
-    <origin xyz="0 0 0" rpy="0 0 0"/>
-  </joint>
-  <!-- ====================== LIDAR ====================== -->
-  <link name="lidar">
-    <visual>
-      <origin xyz="0 0 0" rpy="0 0 0"/>
-      <geometry>
-        <mesh filename="package://robot_description/models/qcar/QCarLidar.stl" scale="0.001 0.001 0.001"/>
-      </geometry>
-      <material name="blue"/>
-    </visual>
-    <collision>
-      <origin xyz="0 0 0" rpy="0 0 0"/>
-      <geometry>
-        <mesh filename="package://robot_description/models/qcar/QCarLidar.stl" scale="0.001 0.001 0.001"/>
-      </geometry>
-    </collision>
-    <inertial>
-      <origin xyz="0 0 0" rpy="0 0 0"/>
-      <mass value="0.1"/>
-      <inertia ixx="0.001" ixy="0" ixz="0" iyy="0.001" iyz="0" izz="0.001"/>
-    </inertial>
-  </link>
-  <joint name="body_lidar_joint" type="fixed">
-    <parent link="base"/>
-    <child link="lidar"/>
-    <origin xyz="-0.01227 -0.00045 0.16152" rpy="0 0 0"/>
-    <axis xyz="0 0 1"/>
-  </joint>
-  <!-- ====================== WHEELS AND HUBS ====================== -->
-  <!-- Front Left Hub -->
-  <link name="hubfl">
-    <visual>
-      <origin xyz="0 0 0" rpy="0 0 0"/>
-      <geometry>
-        <mesh filename="package://robot_description/models/qcar/QCarSteeringHubL.stl" scale="0.001 0.001 0.001"/>
-      </geometry>
-      <material name="orange"/>
-    </visual>
-    <collision>
-      <origin xyz="0 0 0" rpy="0 0 0"/>
-      <geometry>
-        <mesh filename="package://robot_description/models/qcar/QCarSteeringHubL.stl" scale="0.001 0.001 0.001"/>
-      </geometry>
-    </collision>
-    <inertial>
-      <origin xyz="0 0 0" rpy="0 0 0"/>
-      <mass value="0.1"/>
-      <inertia ixx="0.001" ixy="0" ixz="0" iyy="0.001" iyz="0" izz="0.001"/>
-    </inertial>
-  </link>
-  <joint name="base_hubfl_joint" type="revolute">
-    <parent link="base"/>
-    <child link="hubfl"/>
-    <origin xyz="0.1296 0.0559 0.03338" rpy="0 0 0"/>
-    <axis xyz="0 0 1"/>
-    <limit lower="-0.5236" upper="0.5236" effort="300" velocity="2"/>
-    <dynamics damping="0.143" friction="0"/>
-  </joint>
-  <!-- Front Right Hub -->
-  <link name="hubfr">
-    <visual>
-      <origin xyz="0 0 0" rpy="0 0 0"/>
-      <geometry>
-        <mesh filename="package://robot_description/models/qcar/QCarSteeringHubR.stl" scale="0.001 0.001 0.001"/>
-      </geometry>
-      <material name="orange"/>
-    </visual>
-    <collision>
-      <origin xyz="0 0 0" rpy="0 0 0"/>
-      <geometry>
-        <mesh filename="package://robot_description/models/qcar/QCarSteeringHubR.stl" scale="0.001 0.001 0.001"/>
-      </geometry>
-    </collision>
-    <inertial>
-      <origin xyz="0 0 0" rpy="0 0 0"/>
-      <mass value="0.1"/>
-      <inertia ixx="0.001" ixy="0" ixz="0" iyy="0.001" iyz="0" izz="0.001"/>
-    </inertial>
-  </link>
-  <joint name="base_hubfr_joint" type="revolute">
-    <parent link="base"/>
-    <child link="hubfr"/>
-    <origin xyz="0.1296 -0.0559 0.03338" rpy="0 0 0"/>
-    <axis xyz="0 0 1"/>
-    <limit lower="-0.5236" upper="0.5236" effort="300" velocity="2"/>
-    <dynamics damping="0.143" friction="0"/>
-  </joint>
-  <!-- Front Wheels -->
-  <link name="wheelfl">
-    <visual>
-      <origin xyz="0 0 0" rpy="0 0 0"/>
-      <geometry>
-        <mesh filename="package://robot_description/models/qcar/QCarWheel.stl" scale="0.001 0.001 0.001"/>
-      </geometry>
-      <material name="red"/>
-    </visual>
-    <collision>
-      <origin xyz="0 0 0" rpy="0 0 0"/>
-      <geometry>
-        <mesh filename="package://robot_description/models/qcar/QCarWheel.stl" scale="0.001 0.001 0.001"/>
-      </geometry>
-    </collision>
-    <inertial>
-      <origin xyz="0 0 0" rpy="0 0 0"/>
-      <mass value="0.1"/>
-      <inertia ixx="0.001" ixy="0" ixz="0" iyy="0.001" iyz="0" izz="0.001"/>
-    </inertial>
-  </link>
-  <joint name="hubfl_wheelfl_joint" type="continuous">
-    <parent link="hubfl"/>
-    <child link="wheelfl"/>
-    <origin xyz="0 0 0" rpy="0 0 3.14"/>
-    <axis xyz="0 1 0"/>
-  </joint>
-  <link name="wheelfr">
-    <visual>
-      <origin xyz="0 0 0" rpy="0 0 0"/>
-      <geometry>
-        <mesh filename="package://robot_description/models/qcar/QCarWheel.stl" scale="0.001 0.001 0.001"/>
-      </geometry>
-      <material name="orange"/>
-    </visual>
-    <collision>
-      <origin xyz="0 0 0" rpy="0 0 0"/>
-      <geometry>
-        <mesh filename="package://robot_description/models/qcar/QCarWheel.stl" scale="0.001 0.001 0.001"/>
-      </geometry>
-    </collision>
-    <inertial>
-      <origin xyz="0 0 0" rpy="0 0 0"/>
-      <mass value="0.1"/>
-      <inertia ixx="0.001" ixy="0" ixz="0" iyy="0.001" iyz="0" izz="0.001"/>
-    </inertial>
-  </link>
-  <joint name="hubfr_wheelfr_joint" type="continuous">
-    <parent link="hubfr"/>
-    <child link="wheelfr"/>
-    <origin xyz="0 0 0" rpy="0 0 0"/>
-    <axis xyz="0 1 0"/>
-  </joint>
-  <!-- ====================== REAR WHEELS ====================== -->
-  <link name="wheelrl">
-    <visual>
-      <origin xyz="0 0 0" rpy="0 0 0"/>
-      <geometry>
-        <mesh filename="package://robot_description/models/qcar/QCarWheel.stl" scale="0.001 0.001 0.001"/>
-      </geometry>
-      <material name="orange"/>
-    </visual>
-    <collision>
-      <origin xyz="0 0 0" rpy="0 0 0"/>
-      <geometry>
-        <mesh filename="package://robot_description/models/qcar/QCarWheel.stl" scale="0.001 0.001 0.001"/>
-      </geometry>
-    </collision>
-    <inertial>
-      <origin xyz="0 0 0" rpy="0 0 0"/>
-      <mass value="0.1"/>
-      <inertia ixx="0.001" ixy="0" ixz="0" iyy="0.001" iyz="0" izz="0.001"/>
-    </inertial>
-  </link>
-  <joint name="base_wheelrl_joint" type="continuous">
-    <parent link="base"/>
-    <child link="wheelrl"/>
-    <origin xyz="-0.12765 0.0561 0.03338" rpy="0 0 3.14"/>
-    <axis xyz="0 1 0"/>
-  </joint>
-  <link name="wheelrr">
-    <visual>
-      <origin xyz="0 0 0" rpy="0 0 0"/>
-      <geometry>
-        <mesh filename="package://robot_description/models/qcar/QCarWheel.stl" scale="0.001 0.001 0.001"/>
-      </geometry>
-      <material name="red"/>
-    </visual>
-    <collision>
-      <origin xyz="0 0 0" rpy="0 0 0"/>
-      <geometry>
-        <mesh filename="package://robot_description/models/qcar/QCarWheel.stl" scale="0.001 0.001 0.001"/>
-      </geometry>
-    </collision>
-    <inertial>
-      <origin xyz="0 0 0" rpy="0 0 0"/>
-      <mass value="0.1"/>
-      <inertia ixx="0.001" ixy="0" ixz="0" iyy="0.001" iyz="0" izz="0.001"/>
-    </inertial>
-  </link>
-  <joint name="base_wheelrr_joint" type="continuous">
-    <parent link="base"/>
-    <child link="wheelrr"/>
-    <origin xyz="-0.12765 -0.0561 0.03338" rpy="0 0 0"/>
-    <axis xyz="0 1 0"/>
-  </joint>
-  <!-- ====================== CAMERAS ====================== -->
-  <xacro:sensor_d435 name="camera" parent="camera_rgb">
-    <origin xyz="0 0 0" rpy="0 0 0"/>
-  </xacro:sensor_d435>
-  <link name="camera_rgb"/>
-  <joint name="camera_rgb_joint" type="fixed">
-    <parent link="base"/>
-    <child link="camera_rgb"/>
-    <origin xyz="0.081686 0 0.15445" rpy="0 0 0"/>
-  </joint>
-  <joint name="camera_csi_front_joint" type="fixed">
-    <parent link="base"/>
-    <child link="camera_csi_front"/>
-    <origin xyz="0.19236 -0.000475 0.093029" rpy="0 0 0"/>
-  </joint>
-  <link name="camera_csi_front"/>
-  <joint name="camera_csi_right_joint" type="fixed">
-    <parent link="base"/>
-    <child link="camera_csi_right"/>
-    <origin xyz="0.12887 -0.06755 0.093029" rpy="0 0 -1.5708"/>
-  </joint>
-  <link name="camera_csi_right"/>
-  <joint name="camera_csi_back_joint" type="fixed">
-    <parent link="base"/>
-    <child link="camera_csi_back"/>
-    <origin xyz="-0.16669 -0.000578 0.093029" rpy="0 0 -3.1416"/>
-  </joint>
-  <link name="camera_csi_back"/>
-  <joint name="camera_csi_left_joint" type="fixed">
-    <parent link="base"/>
-    <child link="camera_csi_left"/>
-    <origin xyz="0.12784 0.052497 0.093029" rpy="0 0 1.5708"/>
-  </joint>
-  <link name="camera_csi_left"/>
-  <!-- ====================== TRANSMISSIONS ====================== -->
-  <xacro:property name="trans_type" value="transmission_interface/SimpleTransmission"/>
-  <xacro:property name="hw_pos" value="hardware_interface/PositionJointInterface"/>
-  <xacro:property name="hw_eff" value="hardware_interface/EffortJointInterface"/>
-  <xacro:property name="hw_vel" value="hardware_interface/VelocityJointInterface"/>
-  <transmission name="body_lidar_tran">
-    <type>${trans_type}</type>
-    <joint name="body_lidar_joint"><hardwareInterface>${hw_eff}</hardwareInterface></joint>
-    <actuator name="body_lidar_motor"><mechanicalReduction>1</mechanicalReduction></actuator>
-  </transmission>
-  <transmission name="base_hubfl_tran">
-    <type>${trans_type}</type>
-    <joint name="base_hubfl_joint"><hardwareInterface>${hw_pos}</hardwareInterface></joint>
-    <actuator name="base_hubfl_motor"><mechanicalReduction>1</mechanicalReduction></actuator>
-  </transmission>
-  <transmission name="base_hubfr_tran">
-    <type>${trans_type}</type>
-    <joint name="base_hubfr_joint"><hardwareInterface>${hw_pos}</hardwareInterface></joint>
-    <actuator name="base_hubfr_motor"><mechanicalReduction>1</mechanicalReduction></actuator>
-  </transmission>
-  <transmission name="hubfl_wheelfl_tran">
-    <type>${trans_type}</type>
-    <joint name="hubfl_wheelfl_joint"><hardwareInterface>${hw_eff}</hardwareInterface></joint>
-    <actuator name="hubfl_wheelfl_motor"><mechanicalReduction>1</mechanicalReduction></actuator>
-  </transmission>
-  <transmission name="hubfr_wheelfr_tran">
-    <type>${trans_type}</type>
-    <joint name="hubfr_wheelfr_joint"><hardwareInterface>${hw_eff}</hardwareInterface></joint>
-    <actuator name="hubfr_wheelfr_motor"><mechanicalReduction>1</mechanicalReduction></actuator>
-  </transmission>
-  <transmission name="base_wheelrl_tran">
-    <type>${trans_type}</type>
-    <joint name="base_wheelrl_joint"><hardwareInterface>${hw_vel}</hardwareInterface></joint>
-    <actuator name="base_wheelrl_motor"><mechanicalReduction>1</mechanicalReduction></actuator>
-  </transmission>
-  <transmission name="base_wheelrr_tran">
-    <type>${trans_type}</type>
-    <joint name="base_wheelrr_joint"><hardwareInterface>${hw_vel}</hardwareInterface></joint>
-    <actuator name="base_wheelrr_motor"><mechanicalReduction>1</mechanicalReduction></actuator>
-  </transmission>
-  <!-- ====================== GAZEBO PLUGINS ====================== -->
-  <gazebo>
-    <plugin name="gazebo_ros_control" filename="libgazebo_ros_control.so">
-      <robotNamespace>/qcar</robotNamespace>
-    </plugin>
-  </gazebo>
-  <gazebo reference="camera_csi_front">
-    <sensor type="camera" name="front_camera">
-      <update_rate>30.0</update_rate>
-      <camera name="head">
-        <horizontal_fov>2</horizontal_fov>
-        <image>
-          <width>640</width>
-          <height>480</height>
-          <format>R8G8B8</format>
-        </image>
-      </camera>
-      <plugin name="camera_controller" filename="libgazebo_ros_camera.so">
-        <cameraName>qcar/csi_front</cameraName>
-      </plugin>
-    </sensor>
-  </gazebo>
+<robot name="QCar" xmlns:xacro="http://ros.org/wiki/xacro">
+<material name="black">
+<color rgba="0 0 0 1"/>
+</material>
+<material name="blue">
+<color rgba="0 0 0.8 1"/>
+</material>
+<material name="green">
+<color rgba="0 0.8 0 1"/>
+</material>
+<material name="grey">
+<color rgba="0.2 0.2 0.2 1"/>
+</material>
+<material name="orange">
+<color rgba="1.0 0.4235 0.0392 1"/>
+</material>
+<material name="brown">
+<color rgba="0.8706 0.8118 0.7647 1"/>
+</material>
+<material name="red">
+<color rgba="0.8 0 0 1"/>
+</material>
+<material name="white">
+<color rgba="1 1 1 1"/>
+</material>
+<xacro:include filename="$(find realsense2_description)/urdf/_d435.urdf.xacro"/>
+<link name="base">
+<visual>
+<origin xyz="0 0 0" rpy="0 0 0"/>
+<geometry>
+<mesh filename="package://robot_description/models/qcar/QCarBody.stl" scale="0.001 0.001 0.001"/>
+</geometry>
+<material name="white"/>
+</visual>
+<collision>
+<origin xyz="0 0 0" rpy="0 0 0"/>
+<geometry>
+<mesh filename="package://robot_description/models/qcar/QCarBody.stl" scale="0.001 0.001 0.001"/>
+</geometry>
+</collision>
+<inertial>
+<origin xyz="0 0 0" rpy="0 0 0"/>
+<mass value="0.1"/>
+<inertia ixx="0.001" ixy="0" ixz="0" iyy="0.001" iyz="0" izz="0.001"/>
+</inertial>
+</link>
+<link name="base_footprint"/>
+<joint name="base_to_base_footprint" type="fixed">
+<parent link="base"/>
+<child link="base_footprint"/>
+<origin xyz="0 0 0" rpy="0 0 0"/>
+</joint>
+<link name="base_link"/>
+<joint name="base_to_base_link" type="fixed">
+<parent link="base"/>
+<child link="base_link"/>
+<origin xyz="0 0 0" rpy="0 0 0"/>
+</joint>
+<link name="imu_link">
+<inertial>
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
Commit message: mapping works perfectly

File: src/robot_description/urdf/qcar_model.xacro (robot description, xacro)
@@ -92,5 +92,5 @@
 <parent link="base"/>
 <child link="lidar"/>
-<origin xyz="-0.0108 0.0 0.1696" rpy="0 0 1.5708"/>
+<origin xyz="-0.0108 0.0 0.1696" rpy="0 0 1.54"/>
 <axis xyz="0 0 1"/>
 </joint>
